Commit message: Added ar camera support

File: james_description/urdf/james.urdf.xacro (robot description, xacro)
@@ -7,10 +7,10 @@
 	  </plugin>
 	</gazebo>
-	<xacro:property name="box_length" value=".68" />
-	<xacro:property name="box_width" value=".31" />
-	<xacro:property name="box_height" value=".32" />
+	<xacro:property name="box_length" value=".5" />
+	<xacro:property name="box_width" value=".5" />
+	<xacro:property name="box_height" value=".2" />
 	<xacro:property name="wheel_diam" value=".26" />
 	<xacro:property name="wheel_width" value=".075" />
-	<xacro:property name="wheel_axis_offset" value=".20" />
+	<xacro:property name="wheel_axis_offset" value=".10" />
 	<xacro:property name="tail_wheel_diam" value="0.1"/>
 	<xacro:property name="tail_wheel_width" value=".03" />
@@ -160,5 +160,5 @@
 		<origin xyz="${-tail_wheel_diam/2} 0 0" />
 	</joint>
-	<link name="ultrasonic_servo">
+	<link name="camera">
 		<visual>
 			<geometry>
@@ -170,10 +170,7 @@
 		<xacro:cube_inertial origin_xyz="0 0 0" mass="0.01" width="0.01" height="0.03" depth="0.04"/>
 	</link>
-	<gazebo reference="ultrasonic_servo">
-	  	<material>Gazebo/Red</material>
-	</gazebo>
-	<joint name="base_to_ultrasonic" type="fixed">
-		<parent link="base_link" />
-		<child link="ultrasonic_servo" />
+	<joint name="base_to_camera" type="fixed">
+		<parent link="base_link" />
+		<child link="camera" />
 		<origin xyz="0 0 ${box_height/2}" />
 	</joint>
